File: christmas_pcb.kicad_sch (KiCad schematic)
At the start: 42 parts

Commit message: fix errors and use SMT battery
Parts:
- BT1: footprint Battery:BatteryHolder_Keystone_103_1x20mm -> JLCPCB:BAT-TH_BS-8-1
Connections:
- net GND: no longer TP13.1, TP14.1, TP15.1, TP16.1, TP17.1, TP18.1, TP19.1, TP20.1, TP21.1, TP22.1, TP23.1, TP24.1
- new net: TP13.1, TP14.1
- new net: TP16.1, TP19.1
- new net: TP21.1, TP23.1
- new net: TP15.1, TP18.1
- new net: TP17.1, TP20.1
- new net: TP22.1, TP24.1
Changed lines of the file:
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@@
   (junction (at 82.55 101.6) (diameter 0) (color 0 0 0 0)
   )
-  (junction (at 82.55 152.4) (diameter 0) (color 0 0 0 0)
-  )
   (junction (at 95.25 127) (diameter 0) (color 0 0 0 0)
   )
   (junction (at 82.55 69.85) (diameter 0) (color 0 0 0 0)
   )
-  (junction (at 82.55 165.1) (diameter 0) (color 0 0 0 0)
-  )
   (junction (at 95.25 76.2) (diameter 0) (color 0 0 0 0)
   )
   (junction (at 95.25 69.85) (diameter 0) (color 0 0 0 0)
   )
-  (junction (at 82.55 139.7) (diameter 0) (color 0 0 0 0)
-  )
   (junction (at 95.25 95.25) (diameter 0) (color 0 0 0 0)
   )
@@
   (junction (at 92.075 88.9) (diameter 0) (color 0 0 0 0)
   )
-  (junction (at 82.55 146.05) (diameter 0) (color 0 0 0 0)
-  )
   (junction (at 92.075 63.5) (diameter 0) (color 0 0 0 0)
   )
@@
   (junction (at 82.55 82.55) (diameter 0) (color 0 0 0 0)
   )
-  (junction (at 82.55 158.75) (diameter 0) (color 0 0 0 0)
-  )
-  (junction (at 82.55 171.45) (diameter 0) (color 0 0 0 0)
-  )
   (junction (at 92.075 82.55) (diameter 0) (color 0 0 0 0)
   )
@@
     (stroke (width 0) (type default) (color 0 0 0 0))
   )
-  (wire (pts (xy 82.55 139.7) (xy 82.55 146.05))
-    (stroke (width 0) (type default) (color 0 0 0 0))
-  )
   (wire (pts (xy 84.455 107.95) (xy 82.55 107.95))
     (stroke (width 0) (type default) (color 0 0 0 0))
@@
     (stroke (width 0) (type default) (color 0 0 0 0))
   )
-  (wire (pts (xy 82.55 158.75) (xy 82.55 165.1))
-    (stroke (width 0) (type default) (color 0 0 0 0))
-  )
   (wire (pts (xy 92.075 101.6) (xy 95.25 101.6))
     (stroke (width 0) (type default) (color 0 0 0 0))
@@
     (stroke (width 0) (type default) (color 0 0 0 0))
   )
-  (wire (pts (xy 78.74 139.7) (xy 82.55 139.7))
-    (stroke (width 0) (type default) (color 0 0 0 0))
-  )
   (wire (pts (xy 82.55 165.1) (xy 95.25 165.1))
     (stroke (width 0) (type default) (color 0 0 0 0))
   )
-  (wire (pts (xy 82.55 165.1) (xy 82.55 171.45))
-    (stroke (width 0) (type default) (color 0 0 0 0))
-  )
   (wire (pts (xy 92.075 107.95) (xy 95.25 107.95))
     (stroke (width 0) (type default) (color 0 0 0 0))
@@
     (stroke (width 0) (type default) (color 0 0 0 0))
   )
-  (wire (pts (xy 82.55 152.4) (xy 82.55 158.75))
-    (stroke (width 0) (type default) (color 0 0 0 0))
-  )
   (wire (pts (xy 82.55 158.75) (xy 95.25 158.75))
     (stroke (width 0) (type default) (color 0 0 0 0))
@@
   )
   (wire (pts (xy 95.25 127) (xy 95.25 120.65))
-    (stroke (width 0) (type default) (color 0 0 0 0))
-  )
-  (wire (pts (xy 82.55 146.05) (xy 82.55 152.4))
     (stroke (width 0) (type default) (color 0 0 0 0))
   )
@@
     )
   )
-  (global_label "GND" (shape input) (at 78.74 139.7 180) (fields_autoplaced)
-    (effects (font (size 1.27 1.27)) (justify right))
-    (property "Intersheet References" "${INTERSHEET_REFS}" (id 0) (at 72.4564 139.6206 0)
-      (effects (font (size 1.27 1.27)) (justify right) hide)
-    )
-  )
   (global_label "VCC" (shape input) (at 62.865 88.265 0) (fields_autoplaced)
     (effects (font (size 1.27 1.27)) (justify left))
@@
     (property "Reference" "BT1" (id 0) (at 57.277 80.7212 90))
     (property "Value" "Battery_Cell" (id 1) (at 57.277 83.2612 90))
-    (property "Footprint" "Battery:BatteryHolder_Keystone_103_1x20mm" (id 2) (at 56.769 88.265 90)
+    (property "Footprint" "JLCPCB:BAT-TH_BS-8-1" (id 2) (at 56.769 88.265 90)
       (effects (font (size 1.27 1.27)) hide)
     )
@@
   (symbol_instances
     (path "/c37862b7-9046-4331-8425-95e02e416dec"
-      (reference "BT1") (unit 1) (value "Battery_Cell") (footprint "Battery:BatteryHolder_Keystone_103_1x20mm")
+      (reference "BT1") (unit 1) (value "Battery_Cell") (footprint "JLCPCB:BAT-TH_BS-8-1")
     )
     (path "/fb35e3b1-aff6-41a7-9cf0-52694b95edeb"

Commit message: more fixes and footprints
Parts:
- BT1: footprint JLCPCB:BAT-TH_BS-8-1 -> JLCPCB:BAT_BU2032SM-JJ-GTR
Connections:
- net at TP19.1: now also TP20.1; no longer TP16.1
- net at TP21.1: now also TP22.1; no longer TP23.1
- net at TP15.1: now also TP16.1; no longer TP18.1
- net at TP17.1: now also TP18.1; no longer TP20.1
- net at TP24.1: now also TP23.1; no longer TP22.1
Other:
- moved on the sheet: TP16, TP17, TP18, TP19, TP22, TP23
